File: Simulations/nt_psu_filter_freq.kicad_sch (KiCad schematic)
At the start: 22 parts

Commit message: power supply simulations
Parts:
- removed C1, C2, C4, C5, C6, CLoad1, CLoad2: ${SIM.PARAMS}, symbol Device:C
- removed FB1: BLM21PG220SN1, symbol Device:FerriteBead_Small
- removed L1: ${SIM.PARAMS}, symbol Device:L
- removed R1: 1.2, symbol Device:R
- removed R2: 220m, symbol Device:R
- removed RLoad1, RLoad2: 80, symbol Device:R
Other:
- note added: ".tran 1n 50n"
- note added: "a.ac dec 100 10 500Meg"
- note removed: ".ac dec 100 10 500Meg"
