File: Simulations/nt_psu_transient.kicad_sch (KiCad schematic)
At the start: 17 parts, among them K1 DIPxx-1Axx-13x, K2 DIPxx-1Axx-13x, Q1 PMOS

Commit message: psu implementation final
Parts:
- Q1: value PMOS -> DMP2008UFG
- R4: value 10k -> 1k
Connections:
- net VIN: now also D1.1 (K)
- net VGATE: now reaches C4.1, Q1.2 (G), R5.1, R7.2
- net VSUPPLY: now reaches C4.2, L1.1, Q1.1 (D), R1.1
- net VSUPPLY: no longer D1.1 (K)
Other:
- note added: ".ac dec 100 1k 10G"
- note added: "tran 1u 200m"
- note removed: ".tran 1u 20m"
- note removed: "ac dec 100 10 1G"
- moved on the sheet: C1, C2, C3, C4, D1, K1, K2, L1, Q1, R1, R2, R3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
