File: Simulations/nt_psu_transient.kicad_sch (KiCad schematic)
At the start: 17 parts, among them K1 DIPxx-1Axx-13x, K2 DIPxx-1Axx-13x, Q1 DMP2008UFG

Commit message: switch power to 9V
Parts:
- V1: value 5 -> 9
Changed lines of the file:
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@@
       (effects (font (size 1.27 1.27)) (justify left))
     )
-    (property "Value" "5" (at 170.18 117.4392 0)
+    (property "Value" "9" (at 170.18 117.4392 0)
       (effects (font (size 1.27 1.27)) (justify left))
     )

Commit message: fine tuning before layout
Parts:
- removed C3: 2u, symbol Device:C
- removed D1: SMA5.0A, symbol Device:D_Zener
- removed R4: 1k, symbol Device:R
- R1, R2: value 220m -> 100m
- R3: value 250 -> 50
