File: Simulations/nt_psu.kicad_sch (KiCad schematic)
At the start: 17 parts, among them K1 DIPxx-1Axx-13x, K2 DIPxx-1Axx-13x, Q1 DMP2008UFG

Commit message: cleanup and lcsc part numbers
Other:
- note added: ".tran 1u 200m"
- note added: "ac dec 100 1k 10G"
- note removed: ".ac dec 100 1k 10G"
- note removed: "tran 1u 200m"
Changed lines of the file:
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@@
     (effects (font (size 1.27 1.27)) (justify left bottom))
   )
-  (text ".ac dec 100 1k 10G" (at 177.8 173.355 0)
-    (effects (font (size 5 5)) (justify left bottom))
-  )
-  (text "tran 1u 200m" (at 177.8 180.975 0)
-    (effects (font (size 5 5)) (justify left bottom))
+  (text "ac dec 100 1k 10G" (at 180.34 172.085 0)
+    (effects (font (size 2.54 2.54)) (justify left bottom))
+  )
+  (text ".tran 1u 200m" (at 180.34 177.165 0)
+    (effects (font (size 2.54 2.54)) (justify left bottom))
   )
   (label "VIN" (at 120.015 109.22 0) (fields_autoplaced)
@@
       (effects (font (size 1.27 1.27)) hide)
     )
-    (property "Sim.Pins" "1=port1 2=port2" (at 153.035 60.325 0)
-      (effects (font (size 1.27 1.27)) hide)
-    )
-    (property "Sim.Library" "SPICEModels/1274AS-H-4R7N.lib" (at 153.035 60.325 0)
-      (effects (font (size 1.27 1.27)) hide)
-    )
-    (property "Sim.Name" "1274AS-H-4R7N" (at 153.035 60.325 0)
-      (effects (font (size 1.27 1.27)) hide)
-    )
+    (property "Sim.Pins" "1=1 2=2" (at 153.035 60.325 0)
+      (effects (font (size 1.27 1.27)) hide)
+    )
+    (property "Sim.Library" "SPICEModels/104CDMCCDS.lib" (at 153.035 60.325 0)
+      (effects (font (size 1.27 1.27)) hide)
+    )
+    (property "Sim.Name" "104CDMCCDS_4R7MC" (at 153.035 60.325 0)
+      (effects (font (size 1.27 1.27)) hide)
+    )
