File: ComputeModule.kicad_sch (KiCad schematic)
At the start: 4 parts, among them J7 RPi CM4Lite Compatible, J8 RPi CM4Lite Compatible

Commit message: cleanup and lcsc part numbers
Parts:
- J7, J8: value RPi CM4Lite Compatible -> DF40HC(3.0)-100DS; Field5 DF40HC(3.0)-100DS -> (none); LCSC (none) -> C424649

Commit message: fan control and other updates
Parts:
- renumbered J7 to J8, J8 to J9
Connections:
- net FAN_PWM: now reaches J8.38 (GPIO11)

Commit message: more power for output, bigger cap
Connections:
- no-connect marks 123 -> 122

Commit message: switch power to 9V
Connections:
- net +3V3_CM4: no longer names the net of J8.78 (GPIO_VREF(1.8v/3.3v_Input)), J8.84 (+3.3v_(Output)), J8.86 (+3.3v_(Output))

Commit message: fine tuning before layout
Connections:
- net at J8.78 (GPIO_VREF(1.8v/3.3v_Input)), J8.84 (+3.3v_(Output)): no longer J8.86 (+3.3v_(Output))
- no-connect marks 122 -> 123
