File: ComputeModule.kicad_sch (KiCad schematic)
At the start: 4 parts, among them J8 DF40HC(3.0)-100DS, J9 DF40HC(3.0)-100DS

Commit message: switch to 0603 footprints
Parts:
- R15, R22: footprint Resistor_SMD:R_0805_2012Metric_Pad1.20x1.40mm_HandSolder -> Resistor_SMD:R_0603_1608Metric
